File: sbduino-uno.sch (KiCad schematic (older format))
At the start: 53 parts, among them CON1 BARREL_JACK, IC1 ATMEGA328P-AU, P1 USB_B, P2 CONN_01X04, P3 CONN_01X04, P4 CONN_02X03, P5 CONN_01X04, P6 CONN_01X08, P7 CONN_01X10, P8 CONN_01X06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

Commit message: kicad 5
Parts:
- C1, C5, C9: symbol CP_Small -> Device:CP_Small
- C10, C11, C12, C13, C14, C15, C16, C2, C3, C4, C6, C7, C8: symbol C_Small -> Device:C_Small
- CON1: symbol BARREL_JACK -> sbduino-uno-rescue:BARREL_JACK
- D1: symbol D -> Device:D
- D2, D3, D4, D6: symbol Led_Small -> sbduino-uno-rescue:Led_Small
- D5: symbol D_Small -> Device:D_Small
- F1: symbol F_Small -> sbduino-uno-rescue:F_Small
- IC1: symbol ATMEGA328P-A -> sbduino-uno-rescue:ATMEGA328P-A
- P1: symbol USB_B-RESCUE-sbduino-uno -> sbduino-uno-rescue:USB_B-RESCUE-sbduino-uno
- P2, P3, P5, X1: symbol CONN_01X04 -> sbduino-uno-rescue:CONN_01X04
- P4: symbol CONN_02X03 -> sbduino-uno-rescue:CONN_02X03
- P6, P9: symbol CONN_01X08 -> sbduino-uno-rescue:CONN_01X08
- P7: symbol CONN_01X10 -> sbduino-uno-rescue:CONN_01X10
- P8: symbol CONN_01X06 -> sbduino-uno-rescue:CONN_01X06
- Q1: symbol Q_PMOS_GSD -> Device:Q_PMOS_GSD
- R1, R10, R2, R3, R4, R5, R6, R7, R8, R9: symbol R_Small -> Device:R_Small
- SW1: symbol SW_PUSH -> sbduino-uno-rescue:SW_PUSH
- U1: symbol LM358 -> sbduino-uno-rescue:LM358
- U2: symbol NCP1117ST50T3G-RESCUE-sbduino-uno -> sbduino-uno-rescue:NCP1117ST50T3G-RESCUE-sbduino-uno
- U3: symbol CH340G_USB_to_UART -> staticboards:CH340G_USB_to_UART
- U4: symbol LP2985 -> staticboards:LP2985
- Y1, Y2: symbol Crystal_Small -> Device:Crystal_Small
